Commit message: feat: LIDAR pipeline is added

File: simulation/smartcart_ws/install/smartcart_description/share/smartcart_description/urdf/smartcart.urdf.xacro (robot description, xacro)
@@ -147,4 +147,5 @@
     </inertial>
   </link>
+  <!-- CASTER JOINT -->
   <joint name="caster_joint"
          type="fixed">
@@ -153,3 +154,104 @@
     <origin xyz="-0.3 0 0.08"/>
   </joint>
+  <!-- =========================
+       GAZEBO DIFFERENTIAL DRIVE
+       ========================= -->
+  <gazebo>
+    <plugin
+      filename="gz-sim-diff-drive-system"
+      name="gz::sim::systems::DiffDrive">
+      <left_joint>left_wheel_joint</left_joint>
+      <right_joint>right_wheel_joint</right_joint>
+      <wheel_separation>0.7</wheel_separation>
+      <wheel_radius>0.15</wheel_radius>
+      <topic>/cmd_vel</topic>
+      <odom_topic>/wheel/odometry</odom_topic>
+      <frame_id>odom</frame_id>
+      <child_frame_id>base_link</child_frame_id>
+      <odom_publisher_frequency>30</odom_publisher_frequency>
+      <tf_topic>/tf</tf_topic>
+    </plugin>
+  </gazebo>
+  <!-- =========================
+       LIDAR LINK
+       ========================= -->
+  <link name="lidar_link">
+    <visual>
+      <origin xyz="0 0 0" rpy="0 0 0"/>
+      <geometry>
+        <cylinder radius="0.08" length="0.05"/>
+      </geometry>
+      <material name="black"/>
+    </visual>
+    <collision>
+      <origin xyz="0 0 0" rpy="0 0 0"/>
+      <geometry>
+        <cylinder radius="0.08" length="0.05"/>
+      </geometry>
+    </collision>
+    <inertial>
+      <mass value="0.1"/>
+      <inertia
+        ixx="0.0001"
+        ixy="0.0"
+        ixz="0.0"
+        iyy="0.0001"
+        iyz="0.0"
+        izz="0.0001"/>
+    </inertial>
+  </link>
+  <!-- =========================
+       LIDAR FIXED JOINT
+       ========================= -->
+  <joint name="lidar_joint"
+         type="fixed">
+    <parent link="base_link"/>
+    <child link="lidar_link"/>
+    <origin xyz="0.25 0 0.38"
+            rpy="0 0 0"/>
+  </joint>
+  <!-- =========================
+       GAZEBO LIDAR SENSOR
+       ========================= -->
+  <gazebo reference="lidar_link">
+    <sensor
+      name="lidar"
+      type="gpu_lidar">
+      <!-- Gazebo Transport topic -->
+      <topic>/scan</topic>
+      <!-- Sensor frequency -->
+      <update_rate>10</update_rate>
+      <!-- Keep sensor active -->
+      <always_on>true</always_on>
+      <!-- Show rays in Gazebo -->
+      <visualize>true</visualize>
+      <!-- =========================
+           RAY CONFIGURATION
+           ========================= -->
+      <ray>
+        <scan>
+          <horizontal>
+            <samples>360</samples>
+            <resolution>1</resolution>
+            <min_angle>-3.14159</min_angle>
+            <max_angle>3.14159</max_angle>
+          </horizontal>
+          <vertical>
+            <samples>1</samples>
+            <resolution>1</resolution>
+            <min_angle>0</min_angle>
+            <max_angle>0</max_angle>
+          </vertical>
+        </scan>
+        <!-- =========================
+             RANGE
+             ========================= -->
+        <range>
+          <min>0.12</min>
+          <max>10.0</max>
+          <resolution>0.01</resolution>
+        </range>
+      </ray>
+    </sensor>
+  </gazebo>
 </robot>

Commit message: feat: camera module is added

File: simulation/smartcart_ws/install/smartcart_description/share/smartcart_description/urdf/smartcart.urdf.xacro (robot description, xacro)
@@ -147,5 +147,7 @@
     </inertial>
   </link>
-  <!-- CASTER JOINT -->
+  <!-- =========================
+       CASTER JOINT
+       ========================= -->
   <joint name="caster_joint"
          type="fixed">
@@ -218,15 +220,8 @@
       name="lidar"
       type="gpu_lidar">
-      <!-- Gazebo Transport topic -->
       <topic>/scan</topic>
-      <!-- Sensor frequency -->
       <update_rate>10</update_rate>
-      <!-- Keep sensor active -->
       <always_on>true</always_on>
-      <!-- Show rays in Gazebo -->
       <visualize>true</visualize>
-      <!-- =========================
-           RAY CONFIGURATION
-           ========================= -->
       <ray>
         <scan>
@@ -244,7 +239,4 @@
           </vertical>
         </scan>
-        <!-- =========================
-             RANGE
-             ========================= -->
         <range>
           <min>0.12</min>
@@ -255,3 +247,51 @@
     </sensor>
   </gazebo>
+  <!-- =========================
+       CAMERA LINK
+       ========================= -->
+  <link name="camera_link">
+    <visual>
+      <origin xyz="0 0 0" rpy="0 0 0"/>
+      <geometry>
+        <box size="0.12 0.08 0.06"/>
+      </geometry>
+      <material name="black"/>
+    </visual>
+  </link>
+  <!-- =========================
+       CAMERA JOINT
+       ========================= -->
+  <joint name="camera_joint"
+         type="fixed">
+    <parent link="base_link"/>
+    <child link="camera_link"/>
+    <!-- Front-mounted camera -->
+    <origin xyz="0.32 0 0.42"
+            rpy="0 0 0"/>
+  </joint>
+  <!-- =========================
+       GAZEBO CAMERA SENSOR
+       ========================= -->
+  <gazebo reference="camera_link">
+    <sensor
+      name="camera"
+      type="camera">
+      <topic>/camera/image_raw</topic>
+      <update_rate>30</update_rate>
+      <always_on>true</always_on>
+      <visualize>true</visualize>
+      <camera>
+        <horizontal_fov>1.047</horizontal_fov>
+        <image>
+          <width>640</width>
+          <height>480</height>
+          <format>R8G8B8</format>
+        </image>
+        <clip>
+          <near>0.1</near>
+          <far>20.0</far>
+        </clip>
+      </camera>
+    </sensor>
+  </gazebo>
 </robot>
